File: PCB.kicad_sch (KiCad schematic)
At the start: 47 parts, among them J1 USB_C_Receptacle_USB2.0_16P, J10 Conn_01x06_Socket, J11 Conn_01x10_Socket, J2 Conn_01x11_Socket, J3 Conn_01x08_Socket, J4 Conn_01x11_Socket, J5 Conn_01x02_Pin, J6 Conn_01x02_Pin, J7 Conn_01x02_Pin, J8 Conn_01x03_Pin, SW1 SW_Push, SW2 SW_Push, SW3 SW_SPDT_312, U1 TB6612FNG, U4 AMS1117-3.3 (UMW), U6 ESP32-S3-WROOM-1

Commit message: ajout nema17, + debut pcb
Parts:
- removed C4: 10uF(25V/20%), Resistor_SMD:R_0805_2012Metric_Pad1.20x1.40mm_HandSolder, symbol Device:C
- removed F1: Fuse, Fuse:Fuse_1206_3216Metric, symbol Device:Fuse
- removed J10: Conn_01x06_Socket, Connector_PinSocket_2.54mm:PinSocket_1x06_P2.54mm_Vertical, symbol Connector:Conn_01x06_Socket
- removed J11: Conn_01x10_Socket, Connector_PinHeader_2.54mm:PinHeader_1x10_P2.54mm_Vertical, symbol Connector:Conn_01x10_Socket
- removed R11, R9: 10k, Resistor_SMD:R_1206_3216Metric_Pad1.30x1.75mm_HandSolder, symbol Device:R
- removed SW3: SW_SPDT_312, symbol Switch:SW_SPDT_312
- added AO4407A1, AO4407A2: PMOS, Package_SO:SOIC-8-1EP_3.9x4.9mm_P1.27mm_EP2.29x3mm_ThermalVias, symbol Simulation_SPICE:PMOS
- added C11, C17, C3: 100nF, Capacitor_SMD:C_0805_2012Metric_Pad1.18x1.45mm_HandSolder, symbol Device:C_Small
- added C13: 10uF, Capacitor_SMD:CP_Elec_4x5.7, symbol Device:C_Polarized
- added C14, C15, C16: 100uF, Capacitor_SMD:CP_Elec_4x5.7, symbol Device:C
- added J10, J15: Conn_01x02_Pin, Connector_AMASS:AMASS_XT30U-F_1x02_P5.0mm_Vertical, symbol Connector:Conn_01x02_Pin
- added J11, J16, J21, VL0: Conn_01x05_Pin, Connector_PinHeader_2.54mm:PinHeader_1x05_P2.54mm_Vertical, symbol Connector:Conn_01x05_Pin
- added J12, J9: Conn_01x02_Pin, Connector_PinHeader_2.54mm:PinHeader_1x02_P2.54mm_Vertical, symbol Connector:Conn_01x02_Pin
- added J13, J14, J22, MPU1: Conn_01x04_Pin, Connector_PinHeader_2.54mm:PinHeader_1x04_P2.54mm_Vertical, symbol Connector:Conn_01x04_Pin
- added J17, J18, J19, J20, J24, J25, VL1, VL2: Conn_01x03_Pin, Jumper:SolderJumper-3_P1.3mm_Open_Pad1.0x1.5mm, symbol Connector:Conn_01x03_Pin
- added JP1, JP2, JP3, JP4, JP5, JP6: Jumper_2_Open, Connector_PinHeader_2.54mm:PinHeader_1x02_P2.54mm_Vertical, symbol Jumper:Jumper_2_Open
- added Q1: IRF4905, Package_TO_SOT_THT:TO-220-3_Vertical, symbol Transistor_FET:IRF4905
- added R13: 10k, Resistor_SMD:R_1206_3216Metric_Pad1.30x1.75mm_HandSolder, symbol Device:R
- added U10: MCP23008-xSO, Package_SO:SOIC-18W_7.5x11.6mm_P1.27mm, symbol Interface_Expansion:MCP23008-xSO
- added U2, U3: LTC4412xS6, Package_TO_SOT_SMD:TSOT-23-6, symbol Power_Management:LTC4412xS6
- added U5: TB6612FNG, Package_SO:SSOP-24_5.3x8.2mm_P0.65mm, symbol Driver_Motor:TB6612FNG
- added U7, U8, U9: TMC2209_SILENTSTEPSTICK, TMC2209:MODULE_TMC2209_SILENTSTEPSTICK, symbol TMC2209_SILENTSTEPSTICK:TMC2209_SILENTSTEPSTICK
- C6: footprint Capacitor_Tantalum_SMD:CP_EIA-6032-15_Kemet-U_HandSolder -> Capacitor_SMD:CP_Elec_4x5.7
- D1: value ~ -> (none)
- J6: footprint Connector_PinHeader_2.54mm:PinHeader_1x02_P2.54mm_Vertical -> Connector_AMASS:AMASS_XT30U-F_1x02_P5.0mm_Vertical
- R1: footprint Resistor_SMD:R_1206_3216Metric_Pad1.30x1.75mm_HandSolder -> Resistor_SMD:R_0805_3216Metric_Pad1.30x1.75mm_HandSolder
- R5, R6, R7, R8: value 10k -> 4.7k; footprint Resistor_SMD:R_1206_3216Metric_Pad1.30x1.75mm_HandSolder -> Resistor_SMD:R_0805_2012Metric_Pad1.20x1.40mm_HandSolder
Connections:
- net VCC_5VUSB is gone; now on net VCC_5V_USB: J1.A4 (VBUS), J1.A9 (VBUS), J1.B4 (VBUS), J1.B9 (VBUS)
- net in_USB_N is gone; now on net USB_N: J1.A7 (D-), J1.B7 (D-)
- net in_USB_P is gone; now on net USB_P: J1.A6 (D+), J1.B6 (D+)
- net 3V3: now also J3.2 (Pin_2), C17.1, JP1.1 (A), JP2.1 (A), JP3.1 (A), JP4.1 (A), JP5.1 (A), JP6.1 (A), U10.18 (VDD), U10.6 (~{RESET}), U7.2 (VIO), U8.2 (VIO), U9.2 (VIO); no longer J3.1 (Pin_1)
- net CS: now also J3.7 (Pin_7), U6.32 (IO39); no longer J3.5 (Pin_5), U6.30 (IO37)
- net GND: now also J2.10 (Pin_10), J3.1 (Pin_1), J4.2 (Pin_2), J6.1 (Pin_1), C11.2, C13.2, C14.2, C15.2, C16.2, C17.2, C3.2, J10.1 (Pin_1), J11.4 (Pin_4), J15.1 (Pin_1), J16.4 (Pin_4), J21.4 (Pin_4), J9.2 (Pin_2), MPU1.3 (Pin_3), U10.3 (A2), U10.4 (A1), U10.5 (A0), U10.9 (VSS), U2.2 (GND), U2.3 (CTL), U3.2 (GND), U3.3 (CTL), U5.10 (PGND2), U5.18 (GND), U5.3 (PGND1), U5.4 (PGND1), U5.9 (PGND2), U7.1 (GND), U7.7 (GND), U8.1 (GND), U8.7 (GND), U9.1 (GND), U9.7 (GND), VL0.4 (Pin_4); no longer J3.2 (Pin_2)
- net M1_IN1: now also U7.16 (~{EN}), U8.16 (~{EN}), U9.16 (~{EN})
- net MOSI: now also J3.4 (Pin_4); no longer J3.3 (Pin_3)
- net NEOPIXEL: now also U6.4 (IO4); no longer U6.12 (IO8)
- net RST: now also J3.5 (Pin_5), U6.30 (IO37); no longer J3.7 (Pin_7), U6.32 (IO39)
- net SCL1: now also J18.1 (Pin_1), J19.3 (Pin_3), VL1.3 (Pin_3), VL2.3 (Pin_3)
- net SCL2: now also U6.35 (IO42), J18.3 (Pin_3), J19.1 (Pin_1), VL1.1 (Pin_1), VL2.1 (Pin_1); no longer U6.4 (IO4)
- net SCLK: now also J3.3 (Pin_3); no longer J3.4 (Pin_4)
- net SDA1: now also J17.3 (Pin_3), J20.1 (Pin_1), J24.1 (Pin_1), J25.1 (Pin_1)
- net SDA2: now also U6.34 (IO41), J17.1 (Pin_1), J20.3 (Pin_3), J24.3 (Pin_3), J25.3 (Pin_3); no longer U6.5 (IO5)
- net VCC_12V: now also C11.1, C13.1, C14.1, C15.1, C16.1, J10.2 (Pin_2), Q1.2 (D), R13.1, U5.13 (VM2), U5.14 (VM3), U5.24 (VM1), U7.8 (VM), U8.8 (VM), U9.8 (VM)
- net VCC_5V: now also J11.5 (Pin_5), J16.5 (Pin_5), J21.5 (Pin_5), VL0.5 (Pin_5); no longer C12.1, C5.1, D6.1 (VDD), J6.1 (Pin_1), J8.1 (Pin_1), U4.3 (VI)
- net VCC_5V_BUCK: now also AO4407A2.1 (S), AO4407A2.2 (S), AO4407A2.3 (S), J15.2 (Pin_2), U3.1 (VIN)
- net VCC_5V_GLOBAL: now also C12.1, C5.1, D6.1 (VDD), J4.1 (Pin_1), J8.1 (Pin_1), U4.3 (VI), AO4407A1.5 (D), AO4407A1.6 (D), AO4407A1.7 (D), AO4407A1.8 (D), AO4407A1.9 (D), AO4407A2.5 (D), AO4407A2.6 (D), AO4407A2.7 (D), AO4407A2.8 (D), AO4407A2.9 (D), C3.1, J12.1 (Pin_1), MPU1.4 (Pin_4), U2.6 (SENSE), U3.6 (SENSE), U5.19 (STBY), U5.20 (VCC)
- net VCC_5V_USB: now also AO4407A1.1 (S), AO4407A1.2 (S), AO4407A1.3 (S), J12.2 (Pin_2), U2.1 (VIN)
- net M3_IN2: now reaches U6.8 (IO15)
- net M3_IN2: now also U5.22 (AIN2)
- net M4_IN1: now reaches U6.9 (IO16)
- net M4_IN1: now also U5.17 (BIN1)
- net GPIO1_D0_d: now reaches J2.1 (Pin_1)
- net 1V8_OUT: now reaches J2.11 (Pin_11)
- net GPIO1_D1_d: now reaches J2.2 (Pin_2)
- net GPIO1_D2_d: now reaches J2.3 (Pin_3)
- net GPIO1_D3_d: now reaches J2.4 (Pin_4)
- net GPIO1_C6_d: now reaches J2.5 (Pin_5)
- net GPIO1_C7_d: now reaches J2.6 (Pin_6)
- net GPIO0_A4_d: now reaches J2.7 (Pin_7)
- net GPIO4_C0_z: now reaches J2.8 (Pin_8)
- net GPIO4_C1_z: now reaches J2.9 (Pin_9)
- net TEAM_BTN: now reaches J5.1 (Pin_1)
- net TEAM_BTN: now also U10.10 (GP0)
- net GPIO1_C4_d: now reaches J4.10 (Pin_10)
- net GPIO1_C5_d: now reaches J4.11 (Pin_11)
- net 3V3_OUT: now reaches J4.3 (Pin_3)
- net GPIO1_B2_d: now reaches J4.4 (Pin_4)
- net GPIO1_B3_u: now reaches J4.5 (Pin_5)
- net GPIO1_C0_d: now reaches J4.6 (Pin_6)
- net GPIO1_C1_d: now reaches J4.7 (Pin_7)
- net GPIO1_C2_d: now reaches J4.8 (Pin_8)
- net GPIO1_C3_d: now reaches J4.9 (Pin_9)
- net LAUNCHPULL: now reaches J7.1 (Pin_1)
- net LAUNCHPULL: now also U10.11 (GP1)
- net SCLs renamed M4_PWM
- net M4_PWM: now also U5.15 (PWMB)
- net SDAs renamed M3_IN1
- net M3_IN1: now also U5.21 (AIN1)
- net VCC_5Vout renamed VCC_12V_IN
- net VCC_12V_IN: now also Q1.3 (S)
- new net: JP4.2 (B), U8.14 (MS2)
- new net: JP3.2 (B), U8.15 (MS1)
- new net: AO4407A2.4 (G), U3.5 (GATE)
- new net: J16.2 (Pin_2), J21.2 (Pin_2), J25.2 (Pin_2)
- new net: J16.3 (Pin_3), J21.3 (Pin_3), VL2.2 (Pin_2)
- new net: J20.2 (Pin_2), MPU1.1 (Pin_1)
- new net: J19.2 (Pin_2), MPU1.2 (Pin_2)
- new net: JP6.2 (B), U9.14 (MS2)
- new net: AO4407A1.4 (G), U2.5 (GATE)
- new net: J11.3 (Pin_3), VL0.3 (Pin_3), VL1.2 (Pin_2)
- new net: J18.2 (Pin_2), U10.2 (SDA)
- new net: JP2.2 (B), U7.14 (MS2)
- new net: JP1.2 (B), U7.15 (MS1)
- new net: J17.2 (Pin_2), U10.1 (SCL)
- new net: JP5.2 (B), U9.15 (MS1)
- new net: J11.2 (Pin_2), J24.2 (Pin_2), VL0.2 (Pin_2)
- new net BAU+: J9.1 (Pin_1), Q1.1 (G), R13.2
- new net EN1: U10.16 (GP6)
- new net EN2: U10.17 (GP7)
- new net M3+: U5.1 (AO1), U5.2 (AO1)
- new net M3-: U5.5 (AO2), U5.6 (AO2)
- new net M3_PWM: U5.23 (PWMA), U6.5 (IO5)
- new net M4+: U5.11 (BO1), U5.12 (BO1)
- new net M4-: U5.7 (BO2), U5.8 (BO2)
- new net M4_IN2: U5.16 (BIN2), U6.12 (IO8)
- new net MOTORA1: J13.1 (Pin_1), U7.3 (M1B)
- new net MOTORA2: J13.2 (Pin_2), U7.4 (M1A)
- new net MOTORA3: J13.3 (Pin_3), U7.5 (M2A)
- new net MOTORA4: J13.4 (Pin_4), U7.6 (M2B)
- new net MOTORB1: J14.1 (Pin_1), U8.3 (M1B)
- new net MOTORB2: J14.2 (Pin_2), U8.4 (M1A)
- new net MOTORB3: J14.3 (Pin_3), U8.5 (M2A)
- new net MOTORB4: J14.4 (Pin_4), U8.6 (M2B)
- new net MOTORC1: J22.1 (Pin_1), U9.3 (M1B)
- new net MOTORC2: J22.2 (Pin_2), U9.4 (M1A)
- new net MOTORC3: J22.3 (Pin_3), U9.5 (M2A)
- new net MOTORC4: J22.4 (Pin_4), U9.6 (M2B)
- new net XSHUT0: U10.12 (GP2), VL0.1 (Pin_1)
- new net XSHUT1: J11.1 (Pin_1), U10.13 (GP3)
- new net XSHUT2: J16.1 (Pin_1), U10.14 (GP4)
- new net XSHUT3: J21.1 (Pin_1), U10.15 (GP5)
- no-connect marks 5 -> 7
Other:
- note added: "12V & 5V Input"
- note added: "12V for buck"
- note added: "Dual 5V Source"
- note added: "I²C (1)"
- note added: "Luckfox Pico Mini B"
- note added: "MCP23017"
- note added: "N20 Motors 1000RPM & NEMA17 12V"
- note added: "NEMA17"
- note added: "Problème Coupure 12V-5V"
- note added: "battery"
- note added: "for 12V BAU here & add shunt for 5V"
- note added: "only 5V USB ? put BAU here & no shunt"
- note removed: "-ST7789 -ILI9341 -GC9A01"
- note removed: "Auto source"
- note removed: "Fuse"
- note removed: "I²C"
- note removed: "Luckfox"
- note removed: "Mounting Holes"
- note removed: "N20 Motors 1000RPM 12V"
- note removed: "PPTC Fuse 3.5A"
- note removed: "VCC_5Vin -> Fuse -> VCC_5out -> BAU -> VCC_5V"
- moved on the sheet: C1, C10, C5, C6, C7, C8, C9, J2, J4, J5, J7, R5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

Commit message: ajout vcc calc & mise forme pcb
Parts:
- removed C13, C6: 10uF, Capacitor_SMD:CP_Elec_4x5.7, symbol Device:C_Polarized
- removed UART0: Conn_01x04_Pin, Connector_PinHeader_2.54mm:PinHeader_1x04_P2.54mm_Vertical, symbol Connector:Conn_01x04_Pin
- added AS1, AS2: Conn_01x04_Pin, Connector_PinHeader_2.54mm:PinHeader_1x04_P2.54mm_Vertical, symbol Connector:Conn_01x04_Pin
- added C13: 100nF, Capacitor_SMD:C_0805_2012Metric_Pad1.18x1.45mm_HandSolder, symbol Device:C_Small
- added J23, J26: Conn_01x03_Pin, Connector_PinHeader_2.54mm:PinHeader_1x03_P2.54mm_Vertical, symbol Connector:Conn_01x03_Pin
- added J27: Conn_01x02_Pin, Connector_PinHeader_2.54mm:PinHeader_1x02_P2.54mm_Vertical, symbol Connector:Conn_01x02_Pin
- added R14: 220k, Resistor_SMD:R_0805_2012Metric_Pad1.20x1.40mm_HandSolder, symbol Device:R
- added R15: 30k, Resistor_SMD:R_0805_2012Metric_Pad1.20x1.40mm_HandSolder, symbol Device:R
- JP1, JP2, JP3, JP4, JP5, JP6: footprint Connector_PinHeader_2.54mm:PinHeader_1x02_P2.54mm_Vertical -> Jumper:SolderJumper-2_P1.3mm_Open_RoundedPad1.0x1.5mm
Connections:
- net MOTORA1 is gone; now on net M1-: J13.1 (Pin_1), U7.3 (M1B)
- net MOTORA2 is gone; now on net M2-: J13.2 (Pin_2), U7.4 (M1A)
- net MOTORA3 is gone; now on net M2+: J13.3 (Pin_3), U7.5 (M2A)
- net MOTORA4 is gone; now on net M1+: J13.4 (Pin_4), U7.6 (M2B)
- net MOTORB1 is gone; now on net M3-: J14.1 (Pin_1), U8.3 (M1B)
- net MOTORB2 is gone; now on net M4-: J14.2 (Pin_2), U8.4 (M1A)
- net MOTORB3 is gone; now on net M4+: J14.3 (Pin_3), U8.5 (M2A)
- net MOTORB4 is gone; now on net M3+: J14.4 (Pin_4), U8.6 (M2B)
- net EN2: now also U7.16 (~{EN}), U8.16 (~{EN})
- net GND: now also U9.16 (~{EN}), AS1.3 (Pin_3), AS2.3 (Pin_3), C13.2, J23.1 (Pin_1), J26.1 (Pin_1), R15.1
- net M1_IN1: now also U7.10 (STEP); no longer U7.16 (~{EN}), U8.16 (~{EN}), U9.16 (~{EN})
- net M1_IN2: now also U7.9 (DIR)
- net M3_IN1: now also U8.10 (STEP)
- net M3_IN2: now also U8.9 (DIR)
- net SCL1: now also AS1.2 (Pin_2)
- net SCL2: now also AS2.2 (Pin_2)
- net SDA1: now also AS1.1 (Pin_1)
- net SDA2: now also AS2.1 (Pin_1)
- net VCC_12V: now also J27.2 (Pin_2), R14.2
- net VCC_5V: no longer UART1.4 (Pin_4)
- net VCC_5V_GLOBAL: now also UART1.4 (Pin_4), AS1.4 (Pin_4), AS2.4 (Pin_4), J23.2 (Pin_2), J26.2 (Pin_2), J27.1 (Pin_1)
- net VCC_CALC: now reaches U6.23 (IO21)
- net VCC_CALC: now also C13.1, R14.1, R15.2
- net SERVO0: now reaches U6.24 (IO47)
- net SERVO0: now also J23.3 (Pin_3)
- net SERVO1: now reaches U6.25 (IO48)
- net SERVO1: now also J26.3 (Pin_3)
Other:
- note added: "15V, 1A MAX"
- note added: "15V, 3.6A MAX"
- note added: "28V, 2A MAX"
- note added: "30V, 12A MAX"
- note added: "AS5600"
- note added: "Inject 5V in 12V lines WHEN ONLY USB"
- note added: "I²C"
- note added: "Mounting holes"
- note added: "SERVOS"
- note added: "Voltage calculator"
- note added: "read 5V to 27V through ADC"
- note removed: "I²C (1)"
- note removed: "Problème Coupure 12V-5V"
- moved on the sheet: C10, C9, H1, H2, H3, H4, J15, J19, J20, MPU1, R5, R6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

Commit message: fix BAU + bug
Parts:
- removed J12: Conn_01x02_Pin, Connector_PinHeader_2.54mm:PinHeader_1x02_P2.54mm_Vertical, symbol Connector:Conn_01x02_Pin
- removed Q1: IRF4905, Package_TO_SOT_THT:TO-220-3_Vertical, symbol Transistor_FET:IRF4905
- added AO4407A3, AO4407A4: PMOS, Package_SO:SOIC-8-1EP_3.9x4.9mm_P1.27mm_EP2.29x3mm_ThermalVias, symbol Simulation_SPICE:PMOS
- added R16: 10k, Resistor_SMD:R_1206_3216Metric_Pad1.30x1.75mm_HandSolder, symbol Device:R
Connections:
- net 3V3: now also C3.1, C8.1, U1.20 (VCC), U5.20 (VCC)
- net BAU+: now also AO4407A3.4 (G), AO4407A4.4 (G), R16.2
- net EN1: now also U1.19 (STBY), U7.16 (~{EN})
- net EN2: now also U5.19 (STBY); no longer U7.16 (~{EN})
- net VCC_12V: now also AO4407A4.5 (D), AO4407A4.6 (D), AO4407A4.7 (D), AO4407A4.8 (D), AO4407A4.9 (D); no longer R13.1
- net VCC_12V_IN: now also R13.1, AO4407A4.1 (S), AO4407A4.2 (S), AO4407A4.3 (S)
- net VCC_5V_GLOBAL: no longer C3.1, C8.1, U1.19 (STBY), U1.20 (VCC), U5.19 (STBY), U5.20 (VCC)
- net VCC_5V_USB: now also AO4407A3.5 (D), AO4407A3.6 (D), AO4407A3.7 (D), AO4407A3.8 (D), AO4407A3.9 (D); no longer J1.A4 (VBUS), J1.A9 (VBUS), J1.B4 (VBUS), J1.B9 (VBUS)
- new net VCC_5V_USB_IN: AO4407A3.1 (S), AO4407A3.2 (S), AO4407A3.3 (S), J1.A4 (VBUS), J1.A9 (VBUS), J1.B4 (VBUS), J1.B9 (VBUS), R16.1
Other:
- note added: "Inject 5V in 12V lines WHEN ONLY USB CONNECTED"
- note added: "MCP23008"
- note added: "Otherwise BOOM !"
- note removed: "Inject 5V in 12V lines WHEN ONLY USB"
- note removed: "MCP23017"
- note removed: "for 12V BAU here & add shunt for 5V"
- note removed: "only 5V USB ? put BAU here & no shunt"
- moved on the sheet: H1, H2, H3, H4, J9

Commit message: changement driver + debut root pcb
Parts:
- removed C1, C11, C3, C8: 100nF, Capacitor_SMD:C_0805_2012Metric_Pad1.18x1.45mm_HandSolder, symbol Device:C_Small
- removed C14, C15, C16: 100uF, Capacitor_SMD:CP_Elec_4x5.7, symbol Device:C
- removed JP1, JP2, JP3, JP4, JP5, JP6: Jumper_2_Open, Jumper:SolderJumper-2_P1.3mm_Open_RoundedPad1.0x1.5mm, symbol Jumper:Jumper_2_Open
- removed U1, U5: TB6612FNG, Package_SO:SSOP-24_5.3x8.2mm_P0.65mm, symbol Driver_Motor:TB6612FNG
- added C11, C8: 470u, Capacitor_THT:C_Radial_D8.0mm_H11.5mm_P3.50mm, symbol Device:C_Polarized_Small
- added C16, C18, C19, C20: 100nF, Capacitor_SMD:C_0805_2012Metric_Pad1.18x1.45mm_HandSolder, symbol Device:C_Small
- added C3, C4, C6: 100u, Capacitor_THT:C_Radial_D8.0mm_H11.5mm_P3.50mm, symbol Device:C_Polarized_Small
- added J12: Conn_01x02_Pin, Connector_PinHeader_2.54mm:PinHeader_1x02_P2.54mm_Vertical, symbol Connector:Conn_01x02_Pin
- added U1, U5: (no value), Package_SO:SOIC-8_3.9x4.9mm_P1.27mm, symbol Custom:RZ7889
- added UART2: Conn_01x04_Pin, Connector_PinHeader_2.54mm:PinHeader_1x04_P2.54mm_Vertical, symbol Connector:Conn_01x04_Pin
- R14: value 220k -> 180k
- R15: value 30k -> 33k
Connections:
- net M1_PWM is gone; now on net M2_IN1: U6.21 (IO13)
- net M2_PWM is gone; now on net M2_IN2: U6.22 (IO14)
- net M4_IN1 is gone; now on net MS2: U6.9 (IO16)
- net M4_IN2 is gone; now on net DIR2: U6.12 (IO8)
- net EN2: now also U9.16 (~{EN})
- net GND: now also C11.2, C16.2, C19.2, C3.2, C4.2, C6.2, C8.2, U1.3 (GND), U5.3 (GND), UART2.1 (Pin_1); no longer U9.16 (~{EN})
- net M1+: now also C18.1, J12.1 (Pin_1), U1.5 (Fo), U1.6 (Fo); no longer J13.4 (Pin_4), U7.6 (M2B)
- net M1-: now also C18.2, J12.2 (Pin_2), U1.7 (Bo), U1.8 (Bo); no longer J13.1 (Pin_1), U7.3 (M1B)
- net M1_IN1: now also U6.19 (IO11), U1.2 (FI); no longer U6.17 (IO9), U7.10 (STEP)
- net M1_IN2: now also U6.20 (IO12), U1.1 (BI); no longer U6.18 (IO10), U7.9 (DIR)
- net M2+: now also J27.1 (Pin_1), C20.1, U5.5 (Fo), U5.6 (Fo); no longer J13.3 (Pin_3), U7.5 (M2A)
- net M2-: now also J27.2 (Pin_2), C20.2, U5.7 (Bo), U5.8 (Bo); no longer J13.2 (Pin_2), U7.4 (M1A)
- net M2_IN1: now also U5.2 (FI); no longer U6.19 (IO11)
- net M2_IN2: now also U5.1 (BI); no longer U6.20 (IO12)
- net VCC_12V: now also C16.1, C19.1, C3.1, C4.1, C6.1, C8.1, U1.4 (VCC), U5.4 (VCC); no longer J27.2 (Pin_2)
- net VCC_5V_GLOBAL: now also C11.1, UART2.4 (Pin_4); no longer J27.1 (Pin_1)
- net MS2: now reaches U8.14 (MS2)
- net MS2: now also U7.14 (MS2), U9.14 (MS2)
- net MS1: now reaches U8.15 (MS1)
- net MS1: now also U6.8 (IO15), U7.15 (MS1), U9.15 (MS1)
- net STEP3: now reaches U9.10 (STEP)
- net STEP3: now also U6.17 (IO9)
- net DIR3: now reaches U9.9 (DIR)
- net DIR3: now also U6.18 (IO10)
- net GPIO1_D0_d renamed UART3_TX
- net GPIO1_D1_d renamed UART3_RX
- net M3+ renamed MOTORB4
- net M3- renamed MOTORB1
- net M3_IN1 renamed STEP2
- net M3_IN2 renamed DIR2
- net DIR2: no longer U6.8 (IO15)
- net M3_PWM renamed STEP1
- net STEP1: now also U7.10 (STEP)
- net M4+ renamed MOTORB3
- net M4- renamed MOTORB2
- net M4_PWM renamed DIR1
- net DIR1: now also U7.9 (DIR)
- net UART0+ renamed UART0_TX+
- net UART0_TX+: now also UART2.2 (Pin_2)
- net UART0- renamed UART0_RX-
- net UART0_RX-: now also UART2.3 (Pin_3)
- net UART1+ renamed UART1_RX-
- net UART1_RX-: now also U6.11 (IO18); no longer U6.10 (IO17)
- net UART1- renamed UART1_TX+
- net UART1_TX+: now also U6.10 (IO17); no longer U6.11 (IO18)
- new net MOTORA1: J13.1 (Pin_1), U7.3 (M1B)
- new net MOTORA2: J13.2 (Pin_2), U7.4 (M1A)
- new net MOTORA3: J13.3 (Pin_3), U7.5 (M2A)
- new net MOTORA4: J13.4 (Pin_4), U7.6 (M2B)
Other:
- note added: "2x VL53L0X linked together on I2C bus"
- note added: "3-20V, 3A MAX"
- note added: "FOR HUGE CALCULATION ALGO LIKE PATH FINDING VISION"
- note added: "Tof - VL53L0X"
- note added: "cut 12V & 5V from battery"
- note added: "cut 5V USB"
- note added: "input 5V for buck"
- note added: "input battery"
- note added: "output 12V for buck"
- note added: "read 0V to 22.9V through ADC"
- note added: "share same capa"
- note added: "x2 N20 Motors 1000RPM"
- note removed: "12V for buck"
- note removed: "15V, 1A MAX"
- note removed: "15V, 3.6A MAX"
- note removed: "IN1 = HIGH & IN2 = LOW => Forward IN1 = LOW & IN2 = HIGH => Backward IN1 = HIGH & IN2 = HIGH => Brake IN1 = LOW & IN2 = LOW => Coast (free wheel)"
- note removed: "Inject 5V in 12V lines WHEN ONLY USB CONNECTED"
- note removed: "I²C"
- note removed: "N20 Motors 1000RPM & NEMA17 12V"
- note removed: "Otherwise BOOM !"
- note removed: "RX"
- note removed: "TX"
- note removed: "battery"
- note removed: "read 5V to 27V through ADC"
- moved on the sheet: J13, J14, J22, U7, U8, U9

Commit message: suite routage
Connections:
- net VCC_5V is gone; now on net VCC_5V_GLOBAL: J11.5 (Pin_5), J16.5 (Pin_5), J21.5 (Pin_5), VL0.5 (Pin_5)
- net EN1: now also U10.13 (GP3); no longer U10.16 (GP6)
- net EN2: now also U10.10 (GP0); no longer U10.17 (GP7)
- net LAUNCHPULL: now also U10.12 (GP2); no longer U10.11 (GP1)
- net SCL1: now also U6.39 (IO1); no longer U6.38 (IO2)
- net SCL2: now also U6.38 (IO2); no longer U6.35 (IO42)
- net SDA1: now also U6.34 (IO41); no longer U6.39 (IO1)
- net SDA2: now also U6.35 (IO42); no longer U6.34 (IO41)
- net TEAM_BTN: now also U10.11 (GP1); no longer U10.10 (GP0)
- net XSHUT0: now also U10.14 (GP4); no longer U10.12 (GP2)
- net XSHUT1: now also U10.15 (GP5); no longer U10.13 (GP3)
- net XSHUT2: now also U10.16 (GP6); no longer U10.14 (GP4)
- net XSHUT3: now also U10.17 (GP7); no longer U10.15 (GP5)

Commit message: routage
Parts:
- removed AO4407A3: PMOS, Package_SO:SOIC-8-1EP_3.9x4.9mm_P1.27mm_EP2.29x3mm_ThermalVias, symbol Simulation_SPICE:PMOS
- removed J25, VL2: Conn_01x03_Pin, Jumper:SolderJumper-3_P1.3mm_Open_Pad1.0x1.5mm, symbol Connector:Conn_01x03_Pin
- removed R16: 10k, Resistor_SMD:R_1206_3216Metric_Pad1.30x1.75mm_HandSolder, symbol Device:R
Connections:
- net DIR2: now also U6.8 (IO15); no longer U6.12 (IO8)
- net DIR3: now also U6.10 (IO17); no longer U6.18 (IO10)
- net EN1: now also U10.10 (GP0); no longer U10.13 (GP3)
- net EN2: now also U10.13 (GP3); no longer U10.10 (GP0)
- net M1_IN1: now also U6.21 (IO13); no longer U6.19 (IO11)
- net M1_IN2: now also U6.22 (IO14); no longer U6.20 (IO12)
- net M2_IN1: now also U6.19 (IO11); no longer U6.21 (IO13)
- net M2_IN2: now also U6.20 (IO12); no longer U6.22 (IO14)
- net MS1: now also U6.23 (IO21); no longer U6.8 (IO15)
- net MS2: now also U6.24 (IO47); no longer U6.9 (IO16)
- net SCL1: now also U6.38 (IO2); no longer U6.39 (IO1)
- net SCL2: now also U6.39 (IO1); no longer U6.38 (IO2)
- net SERVO0: now also U6.17 (IO9); no longer U6.24 (IO47)
- net SERVO1: now also U6.18 (IO10); no longer U6.25 (IO48)
- net STEP3: now also U6.9 (IO16); no longer U6.17 (IO9)
- net UART1_TX+: now also U6.12 (IO8); no longer U6.10 (IO17)
- net VCC_CALC: now also U6.25 (IO48); no longer U6.23 (IO21)
- net at J16.2 (Pin_2), J21.2 (Pin_2): now also J11.2 (Pin_2), J24.2 (Pin_2), VL0.2 (Pin_2)
- net at J16.3 (Pin_3), J21.3 (Pin_3): now also J11.3 (Pin_3), VL0.3 (Pin_3), VL1.2 (Pin_2)
- net UART3_RX renamed UART3_RX-
- net UART3_TX renamed UART3_TX+
Other:
- note removed: "2x VL53L0X linked together on I2C bus"
- note removed: "cut 5V USB"
- moved on the sheet: H1, H2, H3, H4, J16, J21
